File: designs/CAN_RS485/BeagleBone Comms Cape.sch (EAGLE design)
At the start: 57 parts, among them M1 RED, M2 RED, M3 RED, M4 RED, U4 74LVC1G57, U5 74LVC1G57, U6 74LVC1G57, U7 74LVC1G57

Commit message: Added the revised EAGLE schematics. Also removed two files that were probably not intended to be added as they are lock files in EAGLE.
Parts:
- removed BB.CAPE1: BEAGLEBONE.CAPE.TOP/BOTTOM-PADS, GHI-Solutions:BEAGLEBONE.CAPE.TOP/BOTTOM-PADS
- removed C5, C8, C9: .1uF, GHI-BasicComponents:CAPACITOR-(INCH)-0402
- removed C6, C7: .1uF 50V, GHI-BasicComponents:CAPACITOR-(INCH)-0603
- removed D1, D10, D11, D12, D13, D14, D15, D16, D2, D3, D4, D5, D6, D7, D8, D9: B260A-13-F 60V 2A, GHI-BasicComponents:DIODE-SCHOTTKY-(DIODES)-SMA
- removed M1, M2, M3, M4: RED, GHI-BasicComponents:LED-(INCH)-0805
- removed U1: (no value), GHI-IC:CAT24C32
- removed U2, U3: (no value), GHI-IC:ST-L298-TP(VERSION.A)-W/TV
- removed U4, U5, U6, U7: 74LVC1G57, GHI-IC:74LVC1G57
- added BB.CAPE2: BEAGLEBONE.CAPE.TOP/BOTTOM-PADS, GHI-Solutions:BEAGLEBONE.CAPE.TOP/BOTTOM-PADS
- added IC1: (no value), GHI-IC:CAT24C32
- added IC2: 74LVC1G57, GHI2:1G57-SOT-23-6
- added IC3: MAX13487EESA, GHI3:MAX13487EESA
- added IC4: SN65HVD230, GHI:MCP2551
- added LED1, LED2: (no value), GHI-BasicComponents:LED-(INCH)-0805
- added R11, R13: 1k, GHI-BasicComponents:RESISTOR-(INCH)-0402
- added R12, R14: 330, GHI-BasicComponents:RESISTOR-(INCH)-0402
- added SJ3, SJ4: (no value), GHI-Miscellaneous:SOLDER.JOINT-(INCH)-0402
- added T1, T2: PBSS4350Z 50V 3A, GHI-Transistors:PBSS4350Z
- R10, R9: value DNP(2.2k) -> 75 .125W; device GHI-BasicComponents:RESISTOR-(INCH)-0402 -> GHI-BasicComponents:RESISTOR-(INCH)-0805
- R5, R6: value 1k -> DNP(2.2k)
- R7, R8: value 1k -> 120
Connections:
- removed net M1+: D3.ANODE, D4.CATHODE, U2.OUT2, X1.9
- removed net M1-: D1.ANODE, D2.CATHODE, U2.OUT1, X1.10
- removed net M1.HIGH: BB.CAPE1B.GPIO65, U2.INPUT1, U4.IN0
- removed net M1.LOW: U2.INPUT2, U4.Y
- removed net M1.PWM1.B: BB.CAPE1A.EHRPWM.1B, R1.1, U2.ENABLE.A
- removed net M2+: D11.ANODE, D12.CATHODE, U3.OUT2, X1.7
- removed net M2-: D10.CATHODE, D9.ANODE, U3.OUT1, X1.8
- removed net M2.HIGH: BB.CAPE1B.GPIO46, U3.INPUT1, U5.IN0
- removed net M2.LOW: U3.INPUT2, U5.Y
- removed net M2.PWM1.A: BB.CAPE1A.EHRPWM.1A, R2.1, U3.ENABLE.A
- removed net M3+: D15.ANODE, D16.CATHODE, U3.OUT4, X1.3
- removed net M3-: D13.ANODE, D14.CATHODE, U3.OUT3, X1.4
- removed net M3.HIGH: BB.CAPE1B.GPIO26, U3.INPUT3, U7.IN0
- removed net M3.LOW: U3.INPUT4, U7.Y
- removed net M3.PWM2.B: BB.CAPE1B.EHRPWM.2B, R3.2, U3.ENABLE.B
- removed net M4+: D7.ANODE, D8.CATHODE, U2.OUT4, X1.1
- removed net M4-: D5.ANODE, D6.CATHODE, U2.OUT3, X1.2
- removed net M4.HIGH: BB.CAPE1B.GPIO61, U2.INPUT3, U6.IN0
- removed net M4.LOW: U2.INPUT4, U6.Y
- removed net M4.PWM2.A: BB.CAPE1B.EHRPWM.2A, R4.2, U2.ENABLE.B
- removed net N$3: M1.A, R1.2
- removed net N$6: M4.A, R4.1
- removed net P9.11: BB.CAPE1A.UART4.RXD
- removed net P9.13: BB.CAPE1A.UART4.TXD
- removed net P9.15: BB.CAPE1A.GPIO48
- removed net P9.23: BB.CAPE1A.GPIO49
- removed net P9.24: BB.CAPE1A.UART1.TXD
- removed net P9.26: BB.CAPE1A.UART1.RXD
- removed net P9.34: BB.CAPE1A.AGND.ADC
- removed net P9.35: BB.CAPE1A.AIN6
- removed net P9.36: BB.CAPE1A.AIN5
- removed net VIN: C6.1, C7.1, D1.CATHODE, D11.CATHODE, D13.CATHODE, D15.CATHODE, D3.CATHODE, D5.CATHODE, D7.CATHODE, D9.CATHODE, U2.VS, U3.VS, X1.6
- new net 4-20MA.LOOP.A: BB.CAPE2A.AIN5, R9.2, X1.6
- new net 4-20MA.LOOP.B: BB.CAPE2A.AIN6, R10.2, X1.7
- new net AGND: BB.CAPE2A.AGND.ADC, R10.1, R9.1
- new net CAN.H: IC4.CANH, R8.2, X1.4
- new net CAN.L: IC4.CANL, SJ4.2, X1.5
- new net CAN.RD: BB.CAPE2A.UART1.TXD, IC4.RXD
- new net CAN.TD: BB.CAPE2A.UART1.RXD, IC4.TXD
- new net N$7: LED1.A, R11.2
- new net N$8: LED2.A, R13.2
- new net P8.13: BB.CAPE2B.EHRPWM.2B
- new net P8.14: BB.CAPE2B.GPIO26
- new net P8.16: BB.CAPE2B.GPIO46
- new net P8.18: BB.CAPE2B.GPIO65
- new net P8.19: BB.CAPE2B.EHRPWM.2A
- new net P8.26: BB.CAPE2B.GPIO61
- new net P9.14: BB.CAPE2A.EHRPWM.1A
- new net P9.16: BB.CAPE2A.EHRPWM.1B
- new net RS485.A: IC3.A, SJ3.2, X1.3
- new net RS485.B: IC3.B, R7.2, X1.2
- new net RS485.RX: BB.CAPE2A.UART4.RXD, IC2.Y
- new net RS485.RX.5V: IC2.IN1, IC3.RO
- new net RS485.TX: BB.CAPE2A.UART4.TXD, IC3.DI
- new net SINK.A: BB.CAPE2A.GPIO48, R11.1, R12.1
- new net SINK.A-BASE: R12.2, T1.B
- new net SINK.A-TB: T1.C, X1.8
- new net SINK.B: BB.CAPE2A.GPIO49, R13.1, R14.1
- new net SINK.B-BASE: R14.2, T2.B
- new net SINK.B-TB: T2.C, X1.9
- net +5V: now also BB.CAPE2A.VDD.5V(1), BB.CAPE2A.VDD.5V(2), C4.1, IC3.!RE, IC3.!SHDN, IC3.VCC; no longer BB.CAPE1A.VDD.5V(1), BB.CAPE1A.VDD.5V(2), C8.1, C9.1, U2.VSS, U3.VSS
- net A0: now also IC1.A0, R1.2; no longer R5.2, U1.A0
- net A1: now also IC1.A1, R2.2; no longer R6.2, U1.A1
- net A2: now also IC1.A2, R3.2; no longer R7.2, U1.A2
- net GND: now also BB.CAPE2A.DGND1, BB.CAPE2A.DGND2, BB.CAPE2A.DGND3, BB.CAPE2A.DGND4, BB.CAPE2A.DGND5, BB.CAPE2A.DGND6, BB.CAPE2B.DGND1, BB.CAPE2B.DGND2, IC1.VSS, IC2.GND, IC2.IN0, IC3.GND, IC4.RS, IC4.VSS, LED1.K, LED2.K, R1.1, SJ2.1, T1.E, T2.E, X1.1, X1.10; no longer BB.CAPE1A.DGND1, BB.CAPE1A.DGND2, BB.CAPE1A.DGND3, BB.CAPE1A.DGND4, BB.CAPE1A.DGND5, BB.CAPE1A.DGND6, BB.CAPE1B.DGND1, BB.CAPE1B.DGND2, C5.2, C6.2, C7.2, C8.2, C9.2, D10.ANODE, D12.ANODE, D14.ANODE, D16.ANODE, D2.ANODE, D4.ANODE, D6.ANODE, D8.ANODE, M1.K, M2.K, M3.K, M4.K, R6.1, SJ1.1, U1.VSS, U2.GND1, U2.GND2, U2.GND3, U2.GND4, U2.SENSE.A, U2.SENSE.B, U2.THERMAL.PAD, U3.GND1, U3.GND2, U3.GND3, U3.GND4, U3.SENSE.A, U3.SENSE.B, U3.THERMAL.PAD, U4.GND, U4.IN1, U4.IN2, U5.GND, U5.IN1, U5.IN2, U6.GND, U6.IN1, U6.IN2, U7.GND, U7.IN1, U7.IN2, X1.5
- net N$4: now also R8.1, SJ4.1; no longer M2.A, R2.2
- net N$5: now also R7.1, SJ3.1; no longer M3.A, R3.1
- net P8.10: now also BB.CAPE2B.GPIO68; no longer BB.CAPE1B.GPIO68
- net P8.11: now also BB.CAPE2B.GPIO45; no longer BB.CAPE1B.GPIO45
- net P8.12: now also BB.CAPE2B.GPIO44; no longer BB.CAPE1B.GPIO44
- net P8.15: now also BB.CAPE2B.GPIO47; no longer BB.CAPE1B.GPIO47
- net P8.17: now also BB.CAPE2B.GPIO27; no longer BB.CAPE1B.GPIO27
- net P8.20: now also BB.CAPE2B.MMC1.CMD; no longer BB.CAPE1B.MMC1.CMD
- net P8.21: now also BB.CAPE2B.MMC1.CLK; no longer BB.CAPE1B.MMC1.CLK
- net P8.22: now also BB.CAPE2B.MMC1.DAT5; no longer BB.CAPE1B.MMC1.DAT5
- net P8.23: now also BB.CAPE2B.MMC1.DAT4; no longer BB.CAPE1B.MMC1.DAT4
- net P8.24: now also BB.CAPE2B.MMC1.DAT1; no longer BB.CAPE1B.MMC1.DAT1
- net P8.25: now also BB.CAPE2B.MMC1.DAT0; no longer BB.CAPE1B.MMC1.DAT0
- net P8.27: now also BB.CAPE2B.LCD.VSYNC; no longer BB.CAPE1B.LCD.VSYNC
- net P8.28: now also BB.CAPE2B.LCD.PCLK; no longer BB.CAPE1B.LCD.PCLK
- net P8.29: now also BB.CAPE2B.LCD.HSYNC; no longer BB.CAPE1B.LCD.HSYNC
- net P8.3: now also BB.CAPE2B.MMC1.DAT6; no longer BB.CAPE1B.MMC1.DAT6
- net P8.30: now also BB.CAPE2B.LCD.AC.BIAS; no longer BB.CAPE1B.LCD.AC.BIAS
- net P8.31: now also BB.CAPE2B.LCD.DATA14; no longer BB.CAPE1B.LCD.DATA14
- net P8.32: now also BB.CAPE2B.LCD.DATA15; no longer BB.CAPE1B.LCD.DATA15
- net P8.33: now also BB.CAPE2B.LCD.DATA13; no longer BB.CAPE1B.LCD.DATA13
- net P8.34: now also BB.CAPE2B.LCD.DATA11; no longer BB.CAPE1B.LCD.DATA11
- net P8.35: now also BB.CAPE2B.LCD.DATA12; no longer BB.CAPE1B.LCD.DATA12
- net P8.36: now also BB.CAPE2B.LCD.DATA10; no longer BB.CAPE1B.LCD.DATA10
- net P8.37: now also BB.CAPE2B.LCD.DATA8; no longer BB.CAPE1B.LCD.DATA8
- net P8.38: now also BB.CAPE2B.LCD.DATA9; no longer BB.CAPE1B.LCD.DATA9
- net P8.39: now also BB.CAPE2B.LCD.DATA6; no longer BB.CAPE1B.LCD.DATA6
- net P8.4: now also BB.CAPE2B.MMC1.DAT7; no longer BB.CAPE1B.MMC1.DAT7
- net P8.40: now also BB.CAPE2B.LCD.DATA7; no longer BB.CAPE1B.LCD.DATA7
- net P8.41: now also BB.CAPE2B.LCD.DATA4; no longer BB.CAPE1B.LCD.DATA4
- net P8.42: now also BB.CAPE2B.LCD.DATA5; no longer BB.CAPE1B.LCD.DATA5
- net P8.43: now also BB.CAPE2B.LCD.DATA2; no longer BB.CAPE1B.LCD.DATA2
- net P8.44: now also BB.CAPE2B.LCD.DATA3; no longer BB.CAPE1B.LCD.DATA3
- net P8.45: now also BB.CAPE2B.LCD.DATA0; no longer BB.CAPE1B.LCD.DATA0
- net P8.46: now also BB.CAPE2B.LCD.DATA1; no longer BB.CAPE1B.LCD.DATA1
- net P8.5: now also BB.CAPE2B.MMC1.DAT2; no longer BB.CAPE1B.MMC1.DAT2
- net P8.6: now also BB.CAPE2B.MMC1.DAT3; no longer BB.CAPE1B.MMC1.DAT3
- net P8.7: now also BB.CAPE2B.GPIO66; no longer BB.CAPE1B.GPIO66
- net P8.8: now also BB.CAPE2B.GPIO67; no longer BB.CAPE1B.GPIO67
- net P8.9: now also BB.CAPE2B.GPIO69; no longer BB.CAPE1B.GPIO69
- net P9.10: now also BB.CAPE2A.SYS.RESET#; no longer BB.CAPE1A.SYS.RESET#
- net P9.12: now also BB.CAPE2A.GPIO60; no longer BB.CAPE1A.GPIO60
- net P9.17: now also BB.CAPE2A.SPI0.CS0; no longer BB.CAPE1A.SPI0.CS0
- net P9.18: now also BB.CAPE2A.SPI0.D1; no longer BB.CAPE1A.SPI0.D1
- net P9.21: now also BB.CAPE2A.SPI0.D0; no longer BB.CAPE1A.SPI0.D0
- net P9.22: now also BB.CAPE2A.SPI0.SCK; no longer BB.CAPE1A.SPI0.SCK
- net P9.25: now also BB.CAPE2A.GPIO117; no longer BB.CAPE1A.GPIO117
- net P9.27: now also BB.CAPE2A.GPIO115; no longer BB.CAPE1A.GPIO115
- net P9.28: now also BB.CAPE2A.SPI1.CS0; no longer BB.CAPE1A.SPI1.CS0
- net P9.29: now also BB.CAPE2A.SPI1.D0; no longer BB.CAPE1A.SPI1.D0
- net P9.30: now also BB.CAPE2A.GPIO112; no longer BB.CAPE1A.GPIO112
- net P9.31: now also BB.CAPE2A.SPI1.SCK; no longer BB.CAPE1A.SPI1.SCK
- net P9.32: now also BB.CAPE2A.AVDD.ADC; no longer BB.CAPE1A.AVDD.ADC
- net P9.33: now also BB.CAPE2A.AIN4; no longer BB.CAPE1A.AIN4
- net P9.37: now also BB.CAPE2A.AIN2; no longer BB.CAPE1A.AIN2
- net P9.38: now also BB.CAPE2A.AIN3; no longer BB.CAPE1A.AIN3
- net P9.39: now also BB.CAPE2A.AIN0; no longer BB.CAPE1A.AIN0
- net P9.40: now also BB.CAPE2A.AIN1; no longer BB.CAPE1A.AIN1
- net P9.41: now also BB.CAPE2A.GPIO20; no longer BB.CAPE1A.GPIO20
- net P9.42: now also BB.CAPE2A.ECAPPWM0; no longer BB.CAPE1A.ECAPPWM0
- net P9.9: now also BB.CAPE2A.PWR.BTN; no longer BB.CAPE1A.PWR.BTN
- net SCL: now also BB.CAPE2A.I2C2.SCL, IC1.SCL, R6.1; no longer BB.CAPE1A.I2C2.SCL, R10.1, U1.SCL
- net SDA: now also BB.CAPE2A.I2C2.SDA, IC1.SDA, R5.1; no longer BB.CAPE1A.I2C2.SDA, R9.1, U1.SDA
- net SYS.VOUT: now also BB.CAPE2A.SYS.5V(1), BB.CAPE2A.SYS.5V(2); no longer BB.CAPE1A.SYS.5V(1), BB.CAPE1A.SYS.5V(2)
- net VCC: now also BB.CAPE2A.VDD.3V3(1), BB.CAPE2A.VDD.3V3(2), IC1.VCC, IC2.IN2, IC2.VCC, IC4.VDD, R2.1, R3.1, R4.2, R5.2, R6.2, SJ1.1; no longer BB.CAPE1A.VDD.3V3(1), BB.CAPE1A.VDD.3V3(2), C4.1, C5.1, R10.2, R5.1, R7.1, R8.2, R9.2, SJ2.1, U1.VCC, U4.VCC, U5.VCC, U6.VCC, U7.VCC
- net WP: now also IC1.WP, R4.1; no longer R8.1, U1.WP
Other:
- note added: "CAN and RS485 ICs and Sink transistors"
- note removed: "Motor ICs and Header"
- moved on the sheet: C1, C2, C3, C4, JMP1, R1, R10, R2, R3, R4, R5, R6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
