File: designs/Display18/Display18_Cape.sch (EAGLE design)
At the start: 28 parts, among them T1 3904, X5 SPI-LCD-(1.8IN)

Commit message: Added the revised EAGLE schematics. Also removed two files that were probably not intended to be added as they are lock files in EAGLE.
Parts:
- removed BB.CAPE1: BEAGLEBONE.CAPE.BOTTOM-ONLY-PADS.W/TH, GHI-Solutions:BEAGLEBONE.CAPE.BOTTOM-ONLY-PADS.W/TH
- added BB.CAPE2: BEAGLEBONE.CAPE.BOTTOM-ONLY-PADS, GHI-Solutions:BEAGLEBONE.CAPE.BOTTOM-ONLY-PADS
- added C2, C3: .1uF, GHI-BasicComponents:CAPACITOR-(INCH)-0402
- added C4: 4.7uF, GHI-BasicComponents:CAPACITOR-(INCH)-0603
- added FUD4, FUD5, FUD6: FIDUCIAL, GHI:FIDUCIAL
- added IC2: (no value), GHI-IC:MMA8453Q
- added X6, X7, X8: (no value), GHI2:6MM_TACTILE_SWITCH
- added X9: SPI-LCD-(1.8IN), GHI-Connectors:SPI-LCD-(1.8IN)
- C1: value (none) -> .1uF
- R1, R2: device GHI-BasicComponents:RESISTOR-(INCH)-0603 -> GHI-BasicComponents:RESISTOR-(INCH)-0402
- SJ1, SJ2: device GHI-Miscellaneous:SOLDER.JOINT-(INCH)-0603 -> GHI-Miscellaneous:SOLDER.JOINT-(INCH)-0402
- X5: value SPI-LCD-(1.8IN) -> (none); device GHI-Connectors:SPI-LCD-(1.8IN) -> GHI2:6MM_TACTILE_SWITCH
Connections:
- removed net BTN1: BB.CAPE1B.GPIO44, X1.1, X1.2
- removed net BTN2: BB.CAPE1B.GPIO26, X2.1, X2.2
- removed net BTN3: BB.CAPE1B.GPIO46, X3.1, X3.2
- removed net BTN4: BB.CAPE1B.GPIO65, X4.1, X4.2
- removed net LCD.BACKLIGHT: BB.CAPE1B.GPIO61, R11.2
- removed net LCD.DC(GPIO45): BB.CAPE1B.GPIO45, X5.RS
- removed net LCD.RESET(GPIO86): BB.CAPE1B.LCD.VSYNC, X5.RESET
- removed net LCD.SPI1.CS: BB.CAPE1A.SPI1.CS0, X5.CS
- removed net LCD.SPI1.MOSI: BB.CAPE1A.GPIO112, X5.SDA
- removed net LCD.SPI1.SCK: BB.CAPE1A.SPI1.SCK, X5.SCL
- removed net LED1: BB.CAPE1B.EHRPWM.2A, R1.2
- removed net LED2: BB.CAPE1B.EHRPWM.2B, R2.2
- removed net N$282: LED1.A, R1.1
- removed net N$284: LED2.A, R2.1
- new net ACC.IRQ1(GPIO11): BB.CAPE2B.LCD.DATA15, IC2.INT1
- new net ACC.IRQ2(GPIO81): BB.CAPE2B.LCD.DATA11, IC2.INT2
- new net BTN.1(GPIO87): BB.CAPE2B.LCD.HSYNC, X1.1, X1.2
- new net BTN.2(GPIO86): BB.CAPE2B.LCD.VSYNC, X2.1, X2.2
- new net BTN.3(GPIO89): BB.CAPE2B.LCD.AC.BIAS, X3.1, X3.2
- new net BTN.4(GPIO88): BB.CAPE2B.LCD.PCLK, X4.1, X4.2
- new net BTN.5(GPIO60): BB.CAPE2A.GPIO60, X5.1, X5.2
- new net BTN.6(GPIO67): BB.CAPE2B.GPIO67, X6.1, X6.2
- new net BTN.7(GPIO66): BB.CAPE2B.GPIO66, X7.1, X7.2
- new net BTN.8(GPIO72): BB.CAPE2B.LCD.DATA2, X8.1, X8.2
- new net LCD.BACKLIGHT(TIMER5): BB.CAPE2B.GPIO69, R11.2
- new net LCD.DC(GPIO9): BB.CAPE2B.LCD.DATA13, X9.RS
- new net LCD.RESET(GPIO10): BB.CAPE2B.LCD.DATA14, X9.RESET
- new net LCD.SPI0.CLK: BB.CAPE2A.SPI0.SCK, X9.SCL
- new net LCD.SPI0.CS: BB.CAPE2A.SPI0.CS0, X9.CS
- new net LCD.SPI0.MOSI: BB.CAPE2A.SPI0.D1, X9.SDA
- new net LED1(GPIO8): BB.CAPE2B.LCD.DATA12, LED1.A
- new net LED2(GPIO78): BB.CAPE2B.LCD.DATA8, LED2.A
- new net N$3: LED2.K, R2.2
- new net N$4: LED1.K, R1.2
- new net N$6: C3.1, IC2.BYP
- new net VDD_5V: BB.CAPE2A.VDD.5V(1), BB.CAPE2A.VDD.5V(2)
- net +5V: now also BB.CAPE2A.SYS.5V(1), BB.CAPE2A.SYS.5V(2), X9.LED.A; no longer BB.CAPE1A.SYS.5V(1), BB.CAPE1A.SYS.5V(2), X5.LED.A
- net GND: now also BB.CAPE2A.DGND1, BB.CAPE2A.DGND2, BB.CAPE2A.DGND3, BB.CAPE2A.DGND4, BB.CAPE2A.DGND5, BB.CAPE2A.DGND6, BB.CAPE2B.DGND1, BB.CAPE2B.DGND2, C2.2, C3.2, C4.2, IC2.GND.1, IC2.GND.2, IC2.GND.3, IC2.SA0, R1.1, R2.1, X5.3, X5.4, X6.3, X6.4, X7.3, X7.4, X8.3, X8.4, X9.GND1, X9.GND2, X9.GND3; no longer BB.CAPE1A.DGND1, BB.CAPE1A.DGND2, BB.CAPE1A.DGND3, BB.CAPE1A.DGND4, BB.CAPE1A.DGND5, BB.CAPE1A.DGND6, BB.CAPE1B.DGND1, BB.CAPE1B.DGND2, LED1.K, LED2.K, X5.GND1, X5.GND2, X5.GND3
- net LED.K: now also X9.LED.K; no longer X5.LED.K
- net SCL: now also BB.CAPE2A.I2C2.SCL, IC2.SCL; no longer BB.CAPE1A.I2C2.SCL
- net SDA: now also BB.CAPE2A.I2C2.SDA, IC2.SDA; no longer BB.CAPE1A.I2C2.SDA
- net VCC: now also BB.CAPE2A.VDD.3V3(1), BB.CAPE2A.VDD.3V3(2), C2.1, C4.1, IC1.VCC, IC2.VDD, IC2.VDDIO, X9.VCC1, X9.VCC2; no longer BB.CAPE1A.VDD.3V3(1), BB.CAPE1A.VDD.3V3(2), X5.VCC1, X5.VCC2
Other:
- note added: "------------------------------"
- note added: "1 | 0 | 1 | 0 | A2 | A1 | A0 | R/W"
- note added: "1 | 0 | 1 | 0 | H | H | H | R/W = 0x57"
- note added: "1 | 0 | 1 | 0 | H | H | L | R/W = 0x56"
- note added: "1 | 0 | 1 | 0 | H | L | H | R/W = 0x55"
- note added: "1 | 0 | 1 | 0 | H | L | L | R/W = 0x54"
- note added: "1 | 0 | 1 | 0 | L | H | H | R/W = 0x53"
- note added: "1 | 0 | 1 | 0 | L | H | L | R/W = 0x52"
- note added: "1 | 0 | 1 | 0 | L | L | H | R/W = 0x51"
- note added: "1 | 0 | 1 | 0 | L | L | L | R/W = 0x50"
- note added: "A2"
- note added: "Backlight, Buttons, LEDs, and Screen connector"
- note added: "BeagleBone Headers and EEPROM"
- note added: "Slave Address SA0~ 0011101 :High 0011100 :Low"
- moved on the sheet: C1, IC1, JMP1, LED1, LED2, R1, R10, R11, R2, R3, R4, R5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
