File: designs/Display43/Display50_Cape.sch (EAGLE design)
At the start: 36 parts, among them IC13 FAN5333BSX

Commit message: Added the revised EAGLE schematics. Also removed two files that were probably not intended to be added as they are lock files in EAGLE.
Parts:
- removed IC13: FAN5333BSX, GHI-IC:FAN533X
- removed X1: (no value), GHI-Connectors:10-PIN-(0.5MM-PITCH)-FPC-CONNECTOR
- added 4.3, 5.0: (no value), GHI-Connectors:6-PIN-(0.5MM-PITCH)-FPC-CONNECTOR
- added IC3: (no value), GHI-IC:CAT24C32
- BB.DISPLAY.CAPE-(BEAGLEBONE): value BEAGLEBONE.CAPE.DISPLAY-7.BEAGLEBONE -> BEAGLEBONE.CAPE.DISPLAY-X.BEAGLEBONE; device GHI-Solutions:BEAGLEBONE.CAPE.DISPLAY-7.BEAGLEBONE -> GHI-Solutions:BEAGLEBONE.CAPE.DISPLAY-X.BEAGLEBONE
- BB.DISPLAY.CAPE-(CAPE): value BEAGLEBONE.CAPE.DISPLAY-7.CAPE -> BEAGLEBONE.CAPE.DISPLAY-X.CAPE; device GHI-Solutions:BEAGLEBONE.CAPE.DISPLAY-7.CAPE -> GHI-Solutions:BEAGLEBONE.CAPE.DISPLAY-X.CAPE
- C1: value 10uF -> DNP (10uF)
- C2: value 1uF -> DNP (1uF 50V)
- C5: device rcl:C-USC0805K -> GHI-BasicComponents:CAPACITOR-(INCH)-0805
- D1: value ZHCS400 40V 400mA -> DNP (ZHCS400 40V 400mA)
- D3: value 33V 3W -> DNP (33V 3W)
- IC1: value (none) -> PT4110
- IC2: value (none) -> DNP (FAN5333BSX); device GHI-IC:CAT24C32 -> GHI-IC:FAN533X
- L1: value 10uH -> DNP (10uH)
- R2: value 7.5 -> 20
Connections:
- removed net RESET: TP1.TP, X1.4
- new net WAKE: 4.3.4, 5.0.4, TP1.TP
- net +5V: now also IC2.VIN; no longer IC13.VIN
- net A0: now also IC3.A0; no longer IC2.A0
- net A1: now also IC3.A1; no longer IC2.A1
- net A2: now also IC3.A2; no longer IC2.A2
- net BL+: now also IC2.SW; no longer IC13.SW
- net CAP.TOUCH.IRQ: now also 4.3.5, 5.0.5; no longer X1.5
- net GND: now also 4.3.6, 5.0.6, IC2.GND, IC3.VSS; no longer IC13.GND, IC2.VSS, X1.1, X1.10, X1.9
- net I2C.SCL: now also 4.3.1, 5.0.1, IC3.SCL; no longer IC2.SCL, X1.3
- net I2C.SDA: now also 4.3.2, 5.0.2, IC3.SDA; no longer IC2.SDA, X1.2
- net LCD.BACKLIGHT: now also IC2.SHDN#; no longer IC13.SHDN#
- net LED-: now also IC2.FB; no longer IC13.FB
- net VCC: now also 4.3.3, 5.0.3, IC3.VCC; no longer IC2.VCC, X1.7, X1.8
- net WP: now also IC3.WP; no longer IC2.WP
Other:
- note added: "D3 (the zener diode) is not needed across the LED+ and LED- nodes as it will needlessly cause the LED Driver to heat-up forcing the voltage to stay at 33V without a load. For the FAN5333 driver (315mV FB), change R2 to 7.87 Ohms for 40mA (5 in display) and 21 Ohms for 15mA (4.3 in display) For the PT4110 driver (300mV FB), change R2 to 7.5 Ohms for 40mA (5 in display) and 20 Ohms for 15mA (4.3 in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"
- note added: "This is connected to both IC's Enable Pins"
- note added: "This value should be over 45V."
- moved on the sheet: BB.DISPLAY.CAPE-(BEAGLEBONE)A, BB.DISPLAY.CAPE-(BEAGLEBONE)B, BB.DISPLAY.CAPE-(CAPE)A, BB.DISPLAY.CAPE-(CAPE)B, C1, C2, C3, C4, C5, C6, C7, C8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
