File: designs/Load/Load_Cape.sch (EAGLE design)
At the start: 56 parts, among them T1 PBSS4350Z 50V 3A, T2 PBSS4350Z 50V 3A, T3 PBSS4350Z 50V 3A, T4 PBSS4350Z 50V 3A, T5 PBSS4350Z 50V 3A, T6 PBSS4350Z 50V 3A, T7 PBSS4350Z 50V 3A, T8 PBSS4350Z 50V 3A

Commit message: Added the revised EAGLE schematics. Also removed two files that were probably not intended to be added as they are lock files in EAGLE.
Parts:
- removed X5: (no value), GHI-Connectors:TB-10TERM-150MIL.PITCH
- added FUD4, FUD5, FUD6: FIDUCIAL, GHI:FIDUCIAL
- added X1: (no value), GHI-Connectors:TB-10TERM-150MIL.PITCH
- D1, D11, D13, D15, D3, D5, D7, D9: value (none) -> RED
Connections:
- new net +5V: BB.CAPE1A.SYS.5V(1), BB.CAPE1A.SYS.5V(2)
- new net P8.10: BB.CAPE1B.GPIO68
- new net P8.13: BB.CAPE1B.EHRPWM.2B
- new net P8.14: BB.CAPE1B.GPIO26
- new net P8.16: BB.CAPE1B.GPIO46
- new net P8.18: BB.CAPE1B.GPIO65
- new net P8.19: BB.CAPE1B.EHRPWM.2A
- new net P8.20: BB.CAPE1B.MMC1.CMD
- new net P8.21: BB.CAPE1B.MMC1.CLK
- new net P8.22: BB.CAPE1B.MMC1.DAT5
- new net P8.23: BB.CAPE1B.MMC1.DAT4
- new net P8.24: BB.CAPE1B.MMC1.DAT1
- new net P8.25: BB.CAPE1B.MMC1.DAT0
- new net P8.26: BB.CAPE1B.GPIO61
- new net P8.27: BB.CAPE1B.LCD.VSYNC
- new net P8.28: BB.CAPE1B.LCD.PCLK
- new net P8.29: BB.CAPE1B.LCD.HSYNC
- new net P8.3: BB.CAPE1B.MMC1.DAT6
- new net P8.30: BB.CAPE1B.LCD.AC.BIAS
- new net P8.31: BB.CAPE1B.LCD.DATA14
- new net P8.32: BB.CAPE1B.LCD.DATA15
- new net P8.33: BB.CAPE1B.LCD.DATA13
- new net P8.34: BB.CAPE1B.LCD.DATA11
- new net P8.35: BB.CAPE1B.LCD.DATA12
- new net P8.36: BB.CAPE1B.LCD.DATA10
- new net P8.37: BB.CAPE1B.LCD.DATA8
- new net P8.38: BB.CAPE1B.LCD.DATA9
- new net P8.39: BB.CAPE1B.LCD.DATA6
- new net P8.4: BB.CAPE1B.MMC1.DAT7
- new net P8.40: BB.CAPE1B.LCD.DATA7
- new net P8.41: BB.CAPE1B.LCD.DATA4
- new net P8.42: BB.CAPE1B.LCD.DATA5
- new net P8.43: BB.CAPE1B.LCD.DATA2
- new net P8.44: BB.CAPE1B.LCD.DATA3
- new net P8.45: BB.CAPE1B.LCD.DATA0
- new net P8.46: BB.CAPE1B.LCD.DATA1
- new net P8.5: BB.CAPE1B.MMC1.DAT2
- new net P8.6: BB.CAPE1B.MMC1.DAT3
- new net P8.7: BB.CAPE1B.GPIO66
- new net P8.8: BB.CAPE1B.GPIO67
- new net P8.9: BB.CAPE1B.GPIO69
- new net P9.10: BB.CAPE1A.SYS.RESET#
- new net P9.11: BB.CAPE1A.UART4.RXD
- new net P9.12: BB.CAPE1A.GPIO60
- new net P9.13: BB.CAPE1A.UART4.TXD
- new net P9.14: BB.CAPE1A.EHRPWM.1A
- new net P9.15: BB.CAPE1A.GPIO48
- new net P9.16: BB.CAPE1A.EHRPWM.1B
- new net P9.17: BB.CAPE1A.SPI0.CS0
- new net P9.18: BB.CAPE1A.SPI0.D1
- new net P9.21: BB.CAPE1A.SPI0.D0
- new net P9.22: BB.CAPE1A.SPI0.SCK
- new net P9.23: BB.CAPE1A.GPIO49
- new net P9.24: BB.CAPE1A.UART1.TXD
- new net P9.25: BB.CAPE1A.GPIO117
- new net P9.26: BB.CAPE1A.UART1.RXD
- new net P9.28: BB.CAPE1A.SPI1.CS0
- new net P9.29: BB.CAPE1A.SPI1.D0
- new net P9.31: BB.CAPE1A.SPI1.SCK
- new net P9.32: BB.CAPE1A.AVDD.ADC
- new net P9.33: BB.CAPE1A.AIN4
- new net P9.34: BB.CAPE1A.AGND.ADC
- new net P9.35: BB.CAPE1A.AIN6
- new net P9.36: BB.CAPE1A.AIN5
- new net P9.37: BB.CAPE1A.AIN2
- new net P9.38: BB.CAPE1A.AIN3
- new net P9.39: BB.CAPE1A.AIN0
- new net P9.40: BB.CAPE1A.AIN1
- new net P9.9: BB.CAPE1A.PWR.BTN
- new net VDD_5V: BB.CAPE1A.VDD.5V(1), BB.CAPE1A.VDD.5V(2)
- net GND: now also R17.1, R18.1, X1.9; no longer SJ1.1, SJ2.1, X5.9
- net SINK1.TB: now also X1.8; no longer X5.8
- net SINK2: now also BB.CAPE1A.GPIO20; no longer BB.CAPE1A.GPIO112
- net SINK2.TB: now also X1.7; no longer X5.7
- net SINK3: now also BB.CAPE1A.GPIO112; no longer BB.CAPE1A.GPIO60
- net SINK3.TB: now also X1.6; no longer X5.6
- net SINK4: now also BB.CAPE1A.GPIO115; no longer BB.CAPE1A.GPIO48
- net SINK4.TB: now also X1.5; no longer X5.5
- net SINK5: now also BB.CAPE1B.GPIO44; no longer BB.CAPE1B.GPIO46
- net SINK5.TB: now also X1.4; no longer X5.4
- net SINK6: now also BB.CAPE1B.GPIO45; no longer BB.CAPE1B.GPIO65
- net SINK6.TB: now also X1.3; no longer X5.3
- net SINK7.TB: now also X1.2; no longer X5.2
- net SINK8.TB: now also X1.1; no longer X5.1
- net VCC: now also SJ1.1, SJ2.1; no longer R17.1, R18.1
- net VIN: now also X1.10; no longer X5.10
Other:
- note added: "------------------------------"
- note added: "1 | 0 | 1 | 0 | A2 | A1 | A0 | R/W"
- note added: "1 | 0 | 1 | 0 | H | H | H | R/W = 0x57"
- note added: "1 | 0 | 1 | 0 | H | H | L | R/W = 0x56"
- note added: "1 | 0 | 1 | 0 | H | L | H | R/W = 0x55"
- note added: "1 | 0 | 1 | 0 | H | L | L | R/W = 0x54"
- note added: "1 | 0 | 1 | 0 | L | H | H | R/W = 0x53"
- note added: "1 | 0 | 1 | 0 | L | H | L | R/W = 0x52"
- note added: "1 | 0 | 1 | 0 | L | L | H | R/W = 0x51"
- note added: "1 | 0 | 1 | 0 | L | L | L | R/W = 0x50"
- note added: "A2"
- note added: "BeagleBone Headers and EEPROM"
- moved on the sheet: BB.CAPE1A, BB.CAPE1B, C1, D1, D10, D11, D12, D13, D14, D15, D16, D2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
