File: designs/Motor/Motor_Cape.brd (EAGLE design)
At the start: 71.8 x 58.4 mm, 55 parts, among them M1 RED, M2 RED, M3 RED, M4 RED, U4 74LVC1G57, U5 74LVC1G57, U6 74LVC1G57, U7 74LVC1G57

Commit message: Added the revised EAGLE schematics. Also removed two files that were probably not intended to be added as they are lock files in EAGLE.
Parts:
- added C8, C9: .1uF, GHI-BasicComponents:0402
- moved R6 4.83 mm to (35.2, 18.3), turned to 180 degrees
- moved SJ2 4.83 mm to (30.4, 18.3), turned to 0 degrees
- renumbered X5 to X1
Connections:
- new net P8.10: BB.CAPE1.B8.10, BB.CAPE1.T8.10
- new net P8.11: BB.CAPE1.B8.11, BB.CAPE1.T8.11
- new net P8.12: BB.CAPE1.B8.12, BB.CAPE1.T8.12
- new net P8.15: BB.CAPE1.B8.15, BB.CAPE1.T8.15
- new net P8.17: BB.CAPE1.B8.17, BB.CAPE1.T8.17
- new net P8.20: BB.CAPE1.B8.20, BB.CAPE1.T8.20
- new net P8.21: BB.CAPE1.B8.21, BB.CAPE1.T8.21
- new net P8.22: BB.CAPE1.B8.22, BB.CAPE1.T8.22
- new net P8.23: BB.CAPE1.B8.23, BB.CAPE1.T8.23
- new net P8.24: BB.CAPE1.B8.24, BB.CAPE1.T8.24
- new net P8.25: BB.CAPE1.B8.25, BB.CAPE1.T8.25
- new net P8.27: BB.CAPE1.B8.27, BB.CAPE1.T8.27
- new net P8.28: BB.CAPE1.B8.28, BB.CAPE1.T8.28
- new net P8.29: BB.CAPE1.B8.29, BB.CAPE1.T8.29
- new net P8.3: BB.CAPE1.B8.3, BB.CAPE1.T8.3
- new net P8.30: BB.CAPE1.B8.30, BB.CAPE1.T8.30
- new net P8.31: BB.CAPE1.B8.31, BB.CAPE1.T8.31
- new net P8.32: BB.CAPE1.B8.32, BB.CAPE1.T8.32
- new net P8.33: BB.CAPE1.B8.33, BB.CAPE1.T8.33
- new net P8.34: BB.CAPE1.B8.34, BB.CAPE1.T8.34
- new net P8.35: BB.CAPE1.B8.35, BB.CAPE1.T8.35
- new net P8.36: BB.CAPE1.B8.36, BB.CAPE1.T8.36
- new net P8.37: BB.CAPE1.B8.37, BB.CAPE1.T8.37
- new net P8.38: BB.CAPE1.B8.38, BB.CAPE1.T8.38
- new net P8.39: BB.CAPE1.B8.39, BB.CAPE1.T8.39
- new net P8.4: BB.CAPE1.B8.4, BB.CAPE1.T8.4
- new net P8.40: BB.CAPE1.B8.40, BB.CAPE1.T8.40
- new net P8.41: BB.CAPE1.B8.41, BB.CAPE1.T8.41
- new net P8.42: BB.CAPE1.B8.42, BB.CAPE1.T8.42
- new net P8.43: BB.CAPE1.B8.43, BB.CAPE1.T8.43
- new net P8.44: BB.CAPE1.B8.44, BB.CAPE1.T8.44
- new net P8.45: BB.CAPE1.B8.45, BB.CAPE1.T8.45
- new net P8.46: BB.CAPE1.B8.46, BB.CAPE1.T8.46
- new net P8.5: BB.CAPE1.B8.5, BB.CAPE1.T8.5
- new net P8.6: BB.CAPE1.B8.6, BB.CAPE1.T8.6
- new net P8.7: BB.CAPE1.B8.7, BB.CAPE1.T8.7
- new net P8.8: BB.CAPE1.B8.8, BB.CAPE1.T8.8
- new net P8.9: BB.CAPE1.B8.9, BB.CAPE1.T8.9
- new net P9.10: BB.CAPE1.B9.10, BB.CAPE1.T9.10
- new net P9.11: BB.CAPE1.B9.11, BB.CAPE1.T9.11
- new net P9.12: BB.CAPE1.B9.12, BB.CAPE1.T9.12
- new net P9.13: BB.CAPE1.B9.13, BB.CAPE1.T9.13
- new net P9.15: BB.CAPE1.B9.15, BB.CAPE1.T9.15
- new net P9.17: BB.CAPE1.B9.17, BB.CAPE1.T9.17
- new net P9.18: BB.CAPE1.B9.18, BB.CAPE1.T9.18
- new net P9.21: BB.CAPE1.B9.21, BB.CAPE1.T9.21
- new net P9.22: BB.CAPE1.B9.22, BB.CAPE1.T9.22
- new net P9.23: BB.CAPE1.B9.23, BB.CAPE1.T9.23
- new net P9.24: BB.CAPE1.B9.24, BB.CAPE1.T9.24
- new net P9.25: BB.CAPE1.B9.25, BB.CAPE1.T9.25
- new net P9.26: BB.CAPE1.B9.26, BB.CAPE1.T9.26
- new net P9.27: BB.CAPE1.B9.27, BB.CAPE1.T9.27
- new net P9.28: BB.CAPE1.B9.28, BB.CAPE1.T9.28
- new net P9.29: BB.CAPE1.B9.29, BB.CAPE1.T9.29
- new net P9.30: BB.CAPE1.B9.30, BB.CAPE1.T9.30
- new net P9.31: BB.CAPE1.B9.31, BB.CAPE1.T9.31
- new net P9.32: BB.CAPE1.B9.32, BB.CAPE1.T9.32
- new net P9.33: BB.CAPE1.B9.33, BB.CAPE1.T9.33
- new net P9.34: BB.CAPE1.B9.34, BB.CAPE1.T9.34
- new net P9.35: BB.CAPE1.B9.35, BB.CAPE1.T9.35
- new net P9.36: BB.CAPE1.B9.36, BB.CAPE1.T9.36
- new net P9.37: BB.CAPE1.B9.37, BB.CAPE1.T9.37
- new net P9.38: BB.CAPE1.B9.38, BB.CAPE1.T9.38
- new net P9.39: BB.CAPE1.B9.39, BB.CAPE1.T9.39
- new net P9.40: BB.CAPE1.B9.40, BB.CAPE1.T9.40
- new net P9.41: BB.CAPE1.B9.41, BB.CAPE1.T9.41
- new net P9.42: BB.CAPE1.B9.42, BB.CAPE1.T9.42
- new net P9.9: BB.CAPE1.B9.9, BB.CAPE1.T9.9
- net +5V: now also C8.1, C9.1
- net GND: now also C8.2, C9.2, R6.1; no longer SJ2.1
- net M1.HIGH: now also BB.CAPE1.B8.18, BB.CAPE1.T8.18; no longer BB.CAPE1.B8.8, BB.CAPE1.T8.8
- net M2.HIGH: now also BB.CAPE1.B8.16, BB.CAPE1.T8.16; no longer BB.CAPE1.B8.7, BB.CAPE1.T8.7
- net M3.HIGH: now also BB.CAPE1.B8.14, BB.CAPE1.T8.14; no longer BB.CAPE1.B8.9, BB.CAPE1.T8.9
- net M4.HIGH: now also BB.CAPE1.B8.26, BB.CAPE1.T8.26; no longer BB.CAPE1.B8.10, BB.CAPE1.T8.10
- net VCC: now also SJ2.1; no longer R6.1
Routing:
- net M4.HIGH: track 59.8 -> 46.3 mm
- net M1.HIGH: track 78.0 -> 65.5 mm
- net M2.HIGH: track 70.4 -> 60.5 mm
- net M3.HIGH: track 48.3 -> 43.7 mm
- net P8.8: track 0.00 -> 3.47 mm, vias 0 -> 1
- net P8.6: track 0.00 -> 3.47 mm, vias 0 -> 1
- net P8.46: track 0.00 -> 3.47 mm, vias 0 -> 1
- net P8.44: track 0.00 -> 3.47 mm, vias 0 -> 1
- net P8.42: track 0.00 -> 3.47 mm, vias 0 -> 1
- net P8.40: track 0.00 -> 3.47 mm, vias 0 -> 1
- net P8.4: track 0.00 -> 3.47 mm, vias 0 -> 1
- net P8.38: track 0.00 -> 3.47 mm, vias 0 -> 1
- net P8.36: track 0.00 -> 3.47 mm, vias 0 -> 1
- net P8.34: track 0.00 -> 3.47 mm, vias 0 -> 1
- net P8.32: track 0.00 -> 3.47 mm, vias 0 -> 1
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Other:
- board text added: "A2"
