File: designs/Power/Power_Cape.brd (EAGLE design)
At the start: 71.8 x 58.4 mm, 30 parts, among them IC2 MIC4680-ADJ, IC3 LM1117MP-3.3

Commit message: Added the revised EAGLE schematics. Also removed two files that were probably not intended to be added as they are lock files in EAGLE.
Parts:
- removed C4: 220uF 6.3V B45197A1227K409, rcl:D/7343-31W
- removed D5: STPS140A, GHI:DIODE_SMA
- removed IC3: LM1117MP-3.3, GHI:SOT223
- removed JMP1: JUMPER-(X2), GHI-Headers:JUMPER-(X2)
- removed R17, R18, R19, R20: 1k, GHI-BasicComponents:0402
- removed R21, R22: DNP(2.2k), GHI-BasicComponents:0402
- removed SJ1, SJ2: (no value), GHI-Miscellaneous:SOLDER.JOINT(0402)
- added D1: STPS140A, GHI:DIODE_SMA
- added FUD4, FUD5, FUD6: FIDUCIAL, GHI:FIDUCIAL_40MIL
- C1: value (none) -> 15uF 35V T491D156K035AT; device GHI-BasicComponents:0402 -> rcl:D/7343-31W
- C2: value 15uF 35V T491D156K035AT -> 220uF 6.3V B45197A1227K409
- IC1: value (none) -> LM1117MP-3.3; device GHI-IC:UDFN8,2X3(ON-SEMI) -> GHI:SOT223
- L1: value (none) -> 68uH
- moved C1 37.1 mm to (50.8, 15.4), turned to 90 degrees
- moved IC1 31.8 mm to (32.3, 41.4)
- moved C3 30.6 mm to (43.4, 41.4), turned to 180 degrees
- moved C2 30.3 mm to (21.0, 20.7), turned to 0 degrees
- moved D3 26.5 mm to (21.0, 28.2)
- moved FUD2 3.56 mm to (63.9, 56.0)
- renumbered D4 to D2, X5 to X1
Connections:
- removed net A0: IC1.1, R17.2, SJ1.2
- removed net A1: IC1.2, R18.2, SJ2.2
- removed net A2: IC1.3, R19.2
- removed net SCL: BB.CAPE1.B9.19, BB.CAPE1.T9.19, IC1.6, R22.1
- removed net SDA: BB.CAPE1.B9.20, BB.CAPE1.T9.20, IC1.5, R21.1
- removed net WP: IC1.7, JMP1.1, R20.1
- new net P8.10: BB.CAPE1.B8.10, BB.CAPE1.T8.10
- new net P8.11: BB.CAPE1.B8.11, BB.CAPE1.T8.11
- new net P8.12: BB.CAPE1.B8.12, BB.CAPE1.T8.12
- new net P8.13: BB.CAPE1.B8.13, BB.CAPE1.T8.13
- new net P8.14: BB.CAPE1.B8.14, BB.CAPE1.T8.14
- new net P8.15: BB.CAPE1.B8.15, BB.CAPE1.T8.15
- new net P8.16: BB.CAPE1.B8.16, BB.CAPE1.T8.16
- new net P8.17: BB.CAPE1.B8.17, BB.CAPE1.T8.17
- new net P8.18: BB.CAPE1.B8.18, BB.CAPE1.T8.18
- new net P8.19: BB.CAPE1.B8.19, BB.CAPE1.T8.19
- new net P8.20: BB.CAPE1.B8.20, BB.CAPE1.T8.20
- new net P8.21: BB.CAPE1.B8.21, BB.CAPE1.T8.21
- new net P8.22: BB.CAPE1.B8.22, BB.CAPE1.T8.22
- new net P8.23: BB.CAPE1.B8.23, BB.CAPE1.T8.23
- new net P8.24: BB.CAPE1.B8.24, BB.CAPE1.T8.24
- new net P8.25: BB.CAPE1.B8.25, BB.CAPE1.T8.25
- new net P8.26: BB.CAPE1.B8.26, BB.CAPE1.T8.26
- new net P8.27: BB.CAPE1.B8.27, BB.CAPE1.T8.27
- new net P8.28: BB.CAPE1.B8.28, BB.CAPE1.T8.28
- new net P8.29: BB.CAPE1.B8.29, BB.CAPE1.T8.29
- new net P8.3: BB.CAPE1.B8.3, BB.CAPE1.T8.3
- new net P8.30: BB.CAPE1.B8.30, BB.CAPE1.T8.30
- new net P8.31: BB.CAPE1.B8.31, BB.CAPE1.T8.31
- new net P8.32: BB.CAPE1.B8.32, BB.CAPE1.T8.32
- new net P8.33: BB.CAPE1.B8.33, BB.CAPE1.T8.33
- new net P8.34: BB.CAPE1.B8.34, BB.CAPE1.T8.34
- new net P8.35: BB.CAPE1.B8.35, BB.CAPE1.T8.35
- new net P8.36: BB.CAPE1.B8.36, BB.CAPE1.T8.36
- new net P8.37: BB.CAPE1.B8.37, BB.CAPE1.T8.37
- new net P8.38: BB.CAPE1.B8.38, BB.CAPE1.T8.38
- new net P8.39: BB.CAPE1.B8.39, BB.CAPE1.T8.39
- new net P8.4: BB.CAPE1.B8.4, BB.CAPE1.T8.4
- new net P8.40: BB.CAPE1.B8.40, BB.CAPE1.T8.40
- new net P8.41: BB.CAPE1.B8.41, BB.CAPE1.T8.41
- new net P8.42: BB.CAPE1.B8.42, BB.CAPE1.T8.42
- new net P8.43: BB.CAPE1.B8.43, BB.CAPE1.T8.43
- new net P8.44: BB.CAPE1.B8.44, BB.CAPE1.T8.44
- new net P8.45: BB.CAPE1.B8.45, BB.CAPE1.T8.45
- new net P8.46: BB.CAPE1.B8.46, BB.CAPE1.T8.46
- new net P8.5: BB.CAPE1.B8.5, BB.CAPE1.T8.5
- new net P8.6: BB.CAPE1.B8.6, BB.CAPE1.T8.6
- new net P8.7: BB.CAPE1.B8.7, BB.CAPE1.T8.7
- new net P8.8: BB.CAPE1.B8.8, BB.CAPE1.T8.8
- new net P8.9: BB.CAPE1.B8.9, BB.CAPE1.T8.9
- new net P9.11: BB.CAPE1.B9.11, BB.CAPE1.T9.11
- new net P9.12: BB.CAPE1.B9.12, BB.CAPE1.T9.12
- new net P9.13: BB.CAPE1.B9.13, BB.CAPE1.T9.13
- new net P9.14: BB.CAPE1.B9.14, BB.CAPE1.T9.14
- new net P9.15: BB.CAPE1.B9.15, BB.CAPE1.T9.15
- new net P9.16: BB.CAPE1.B9.16, BB.CAPE1.T9.16
- new net P9.17: BB.CAPE1.B9.17, BB.CAPE1.T9.17
- new net P9.18: BB.CAPE1.B9.18, BB.CAPE1.T9.18
- new net P9.19: BB.CAPE1.B9.19, BB.CAPE1.T9.19
- new net P9.20: BB.CAPE1.B9.20, BB.CAPE1.T9.20
- new net P9.21: BB.CAPE1.B9.21, BB.CAPE1.T9.21
- new net P9.22: BB.CAPE1.B9.22, BB.CAPE1.T9.22
- new net P9.23: BB.CAPE1.B9.23, BB.CAPE1.T9.23
- new net P9.24: BB.CAPE1.B9.24, BB.CAPE1.T9.24
- new net P9.25: BB.CAPE1.B9.25, BB.CAPE1.T9.25
- new net P9.26: BB.CAPE1.B9.26, BB.CAPE1.T9.26
- new net P9.27: BB.CAPE1.B9.27, BB.CAPE1.T9.27
- new net P9.28: BB.CAPE1.B9.28, BB.CAPE1.T9.28
- new net P9.29: BB.CAPE1.B9.29, BB.CAPE1.T9.29
- new net P9.30: BB.CAPE1.B9.30, BB.CAPE1.T9.30
- new net P9.31: BB.CAPE1.B9.31, BB.CAPE1.T9.31
- new net P9.32: BB.CAPE1.B9.32, BB.CAPE1.T9.32
- new net P9.33: BB.CAPE1.B9.33, BB.CAPE1.T9.33
- new net P9.34: BB.CAPE1.B9.34, BB.CAPE1.T9.34
- new net P9.35: BB.CAPE1.B9.35, BB.CAPE1.T9.35
- new net P9.36: BB.CAPE1.B9.36, BB.CAPE1.T9.36
- new net P9.37: BB.CAPE1.B9.37, BB.CAPE1.T9.37
- new net P9.38: BB.CAPE1.B9.38, BB.CAPE1.T9.38
- new net P9.39: BB.CAPE1.B9.39, BB.CAPE1.T9.39
- new net P9.40: BB.CAPE1.B9.40, BB.CAPE1.T9.40
- new net P9.41: BB.CAPE1.B9.41, BB.CAPE1.T9.41
- new net P9.42: BB.CAPE1.B9.42, BB.CAPE1.T9.42
- net +5V: now also D3.K, IC1.3; no longer D5.K, IC3.3
- net 5VOUT.B: now also C2.+, D3.A; no longer C3.+, D5.A
- net GND: now also C1.-, IC1.1; no longer C1.2, C4.-, IC1.4, IC3.1, JMP1.2, SJ1.1, SJ2.1
- net REGULATED.3V3: now also C3.+, IC1.2, IC1.4; no longer C4.+, IC3.2, IC3.4
- net VCC: no longer C1.1, IC1.8, R17.1, R18.1, R19.1, R20.2, R21.2, R22.2
- net VIN: now also C1.+, D1.A; no longer C2.+, D3.A
- net VIN.K: now also D1.K; no longer D3.K
Routing:
- net SCL: track 29.1 -> 0.00 mm, vias 3 -> 0
- net SDA: track 24.9 -> 0.00 mm, vias 3 -> 0
- net WP: track 17.4 -> 0.00 mm, vias 1 -> 0
- net A0: track 6.25 -> 0.00 mm
- net A1: track 5.82 -> 0.00 mm
- net GND: track 7.55 -> 2.84 mm, vias 30 -> 26
- net P8.8: track 0.00 -> 3.47 mm, vias 0 -> 1
- net P8.6: track 0.00 -> 3.47 mm, vias 0 -> 1
- net P8.46: track 0.00 -> 3.47 mm, vias 0 -> 1
- net P8.44: track 0.00 -> 3.47 mm, vias 0 -> 1
- net P8.42: track 0.00 -> 3.47 mm, vias 0 -> 1
- net P8.40: track 0.00 -> 3.47 mm, vias 0 -> 1
- net P8.4: track 0.00 -> 3.47 mm, vias 0 -> 1
- net P8.38: track 0.00 -> 3.47 mm, vias 0 -> 1
- net P8.36: track 0.00 -> 3.47 mm, vias 0 -> 1
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Other:
- board text added: "A2"
- board text removed: "A0"
- board text removed: "A1"
- board text removed: "EEPROM WP"
