File: designs/Relay/Relay_Cape.sch (EAGLE design)
At the start: 51 parts, among them T1 3904, T2 3904, T3 3904, T4 3904, X1 RELAY_SINGLE_POLE_DOUBLE_THROW, X2 RELAY_SINGLE_POLE_DOUBLE_THROW, X3 RELAY_SINGLE_POLE_DOUBLE_THROW, X4 RELAY_SINGLE_POLE_DOUBLE_THROW

Commit message: Added the revised EAGLE schematics. Also removed two files that were probably not intended to be added as they are lock files in EAGLE.
Parts:
- added FUD4, FUD5, FUD6: FIDUCIAL, GHI:FIDUCIAL
- R1, R2, R3, R4, R5, R6, R7, R8: device GHI-BasicComponents:RESISTOR-(INCH)-0603 -> GHI-BasicComponents:RESISTOR-(INCH)-0402
Connections:
- net GND: now also R11.1, R12.1; no longer SJ1.1, SJ2.1
- net RELAY1: now also BB.CAPE1A.GPIO20; no longer BB.CAPE1A.GPIO112
- net RELAY2: now also BB.CAPE1A.ECAPPWM0; no longer BB.CAPE1A.GPIO115
- net RELAY3: now also BB.CAPE1A.GPIO112; no longer BB.CAPE1A.GPIO117
- net RELAY4: now also BB.CAPE1A.GPIO115; no longer BB.CAPE1A.GPIO49
- net VCC: now also SJ1.1, SJ2.1; no longer R11.1, R12.1
Other:
- note added: "------------------------------"
- note added: "1 | 0 | 1 | 0 | A2 | A1 | A0 | R/W"
- note added: "1 | 0 | 1 | 0 | H | H | H | R/W = 0x57"
- note added: "1 | 0 | 1 | 0 | H | H | L | R/W = 0x56"
- note added: "1 | 0 | 1 | 0 | H | L | H | R/W = 0x55"
- note added: "1 | 0 | 1 | 0 | H | L | L | R/W = 0x54"
- note added: "1 | 0 | 1 | 0 | L | H | H | R/W = 0x53"
- note added: "1 | 0 | 1 | 0 | L | H | L | R/W = 0x52"
- note added: "1 | 0 | 1 | 0 | L | L | H | R/W = 0x51"
- note added: "1 | 0 | 1 | 0 | L | L | L | R/W = 0x50"
- note added: "A2"
- note added: "BeagleBone Headers and EEPROM"
- note added: "Relays and Header"
- moved on the sheet: BB.CAPE1A, BB.CAPE1B, C1, C2, C3, C4, C5, C6, C7, C8, C9, D1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
