File: designs/Servo/Servo_Cape.sch (EAGLE design)
At the start: 22 parts, among them IC1 LM1117MP-3.3, IC2 MIC4680-ADJ

Commit message: Added the revised EAGLE schematics. Also removed two files that were probably not intended to be added as they are lock files in EAGLE.
Parts:
- removed 3V3, 5V: RED, GHI-BasicComponents:LED-(INCH)-0805
- removed BB.CAPE1: BEAGLEBONE.CAPE.TOP/BOTTOM-PADS, GHI-Solutions:BEAGLEBONE.CAPE.TOP/BOTTOM-PADS
- removed C3: 220uF 6.3V B45197A1227K409, rcl:CPOL-USD/7343-31W
- removed D1, D3: STPS140A, GHI:DIODE_SMA
- removed D2: B130, GHI:DIODE_SMA
- removed IC1: LM1117MP-3.3, GHI:LM1117
- removed IC2: MIC4680-ADJ, GHI:MIC4680
- removed L1: 68uH, GHI-BasicComponents:UP2B-XXX
- added BB.CAPE2: BEAGLEBONE.CAPE.TOP/BOTTOM-PADS, GHI-Solutions:BEAGLEBONE.CAPE.TOP/BOTTOM-PADS
- added IN1, IN2, IN3, IN4, IN5, IN6, S1, S10, S11, S12, S13, S14, S15, S16, S2, S3, S4, S5, S6, S7, S8, S9: (no value), GHI-Headers:1X3-(INCH)-0.1-TH-(35-MIL.DIA)
- added JMP1: JUMPER-(X2), GHI-Headers:JUMPER-(X2)
- added R10, R4, R5, R6, R7, R8, R9: 1k, GHI-BasicComponents:RESISTOR-(INCH)-0402
- added R11, R12: DNP(2.2k), GHI-BasicComponents:RESISTOR-(INCH)-0402
- added SJ1, SJ2, SJ3, SJ4, SJ5, SJ6, SJ7, SJ8: (no value), GHI-Miscellaneous:SOLDER.JOINT-(INCH)-0402
- added U1: CAT24C32, GHI-IC:CAT24C32
- added U2: PCA9685(TSSOP), GHI-IC:PCA9685(TSSOP)
- added X2: (no value), GHI-Headers:1X2-(INCH)-0.1-TH-(35-MIL.DIA)
- C1: value 15uF 35V T491D156K035AT -> .1uF; device rcl:CPOL-USD/7343-31W -> GHI-BasicComponents:CAPACITOR-(INCH)-0402
- C2: value 220uF 6.3V B45197A1227K409 -> .1uF; device rcl:CPOL-USD/7343-31W -> GHI-BasicComponents:CAPACITOR-(INCH)-0402
- X1: value (none) -> TB-2TERM-5MM.PITCH; device GHI-Connectors:TB-10TERM-150MIL.PITCH -> GHI-Connectors:TB-2TERM-5MM.PITCH
Connections:
- removed net 5VOUT.A: D2.K, IC2.SW, L1.1
- removed net 5VOUT.B: C2.+, D3.A, IC2.FB, L1.2
- removed net N$3: 5V.A, R2.2
- removed net N$36: 3V3.A, R3.2
- removed net P8.10: BB.CAPE1B.GPIO68
- removed net P8.11: BB.CAPE1B.GPIO45
- removed net P8.12: BB.CAPE1B.GPIO44
- removed net P9.19: BB.CAPE1A.I2C2.SCL
- removed net P9.20: BB.CAPE1A.I2C2.SDA
- removed net P9.27: BB.CAPE1A.GPIO115
- removed net P9.30: BB.CAPE1A.GPIO112
- removed net P9.41: BB.CAPE1A.GPIO20
- removed net P9.42: BB.CAPE1A.ECAPPWM0
- removed net PWR.BTN: BB.CAPE1A.PWR.BTN, X1.3
- removed net REG.SHUTDOWN: IC2.SHDN, R1.1, X1.8
- removed net REGULATED.3V3: C3.+, IC1.VOUT1, IC1.VOUT2, R3.1, X1.7
- removed net SYS.RESET#: BB.CAPE1A.SYS.RESET#, X1.2
- removed net SYS.VOUT: BB.CAPE1A.SYS.5V(1), BB.CAPE1A.SYS.5V(2), X1.4
- removed net VIN.K: D1.K, IC2.IN
- new net A0: R7.2, SJ1.2, U1.A0
- new net A1: R8.2, SJ2.2, U1.A1
- new net A2: R9.2, U1.A2
- new net IN1: BB.CAPE2B.GPIO44, IN1.3
- new net IN2: BB.CAPE2B.GPIO45, IN2.3
- new net IN3: BB.CAPE2A.GPIO112, IN3.3
- new net IN4: BB.CAPE2A.GPIO115, IN4.3
- new net IN5: BB.CAPE2A.GPIO20, IN5.3
- new net IN6: BB.CAPE2A.ECAPPWM0, IN6.3
- new net P9.10: BB.CAPE2A.SYS.RESET#
- new net P9.9: BB.CAPE2A.PWR.BTN
- new net PWM0: S1.3, U2.LED0
- new net PWM1: S2.3, U2.LED1
- new net PWM10: S11.3, U2.LED10
- new net PWM11: S12.3, U2.LED11
- new net PWM12: S13.3, U2.LED12
- new net PWM13: S14.3, U2.LED13
- new net PWM14: S15.3, U2.LED14
- new net PWM15: S16.3, U2.LED15
- new net PWM2: S3.3, U2.LED2
- new net PWM3: S4.3, U2.LED3
- new net PWM4: S5.3, U2.LED4
- new net PWM5: S6.3, U2.LED5
- new net PWM6: S7.3, U2.LED6
- new net PWM7: S8.3, U2.LED7
- new net PWM8: S9.3, U2.LED8
- new net PWM9: S10.3, U2.LED9
- new net SCL: BB.CAPE2A.I2C2.SCL, R12.1, U1.SCL, U2.SCL
- new net SDA: BB.CAPE2A.I2C2.SDA, R11.1, U1.SDA, U2.SDA
- new net SERVO.ENABLE: BB.CAPE2B.GPIO68, U2.OE#
- new net U2.A0: R1.2, SJ3.2, U2.A0
- new net U2.A1: R2.2, SJ4.2, U2.A1
- new net U2.A2: R3.2, SJ5.2, U2.A2
- new net U2.A3: R4.2, SJ6.2, U2.A3
- new net U2.A4: R5.2, SJ7.2, U2.A4
- new net U2.A5: R6.2, SJ8.2, U2.A5
- new net VOUT: BB.CAPE2A.SYS.5V(1), BB.CAPE2A.SYS.5V(2), X2.2
- new net WP: JMP1.1, R10.1, U1.WP
- net +5V: now also BB.CAPE2A.VDD.5V(1), BB.CAPE2A.VDD.5V(2); no longer BB.CAPE1A.VDD.5V(1), BB.CAPE1A.VDD.5V(2), D3.K, IC1.VIN, R2.1, X1.6
- net GND: now also BB.CAPE2A.DGND1, BB.CAPE2A.DGND2, BB.CAPE2A.DGND3, BB.CAPE2A.DGND4, BB.CAPE2A.DGND5, BB.CAPE2A.DGND6, BB.CAPE2B.DGND1, BB.CAPE2B.DGND2, C1.2, C2.2, IN1.1, IN2.1, IN3.1, IN4.1, IN5.1, IN6.1, JMP1.2, R7.1, R8.1, S1.1, S10.1, S11.1, S12.1, S13.1, S14.1, S15.1, S16.1, S2.1, S3.1, S4.1, S5.1, S6.1, S7.1, S8.1, S9.1, SJ3.1, SJ4.1, SJ5.1, SJ6.1, SJ7.1, SJ8.1, U1.VSS, U2.EXTCLK, U2.VSS, X1.2, X2.1; no longer 3V3.K, 5V.K, BB.CAPE1A.DGND1, BB.CAPE1A.DGND2, BB.CAPE1A.DGND3, BB.CAPE1A.DGND4, BB.CAPE1A.DGND5, BB.CAPE1A.DGND6, BB.CAPE1B.DGND1, BB.CAPE1B.DGND2, C1.-, C2.-, C3.-, D2.A, IC1.GND, IC2.GND1, IC2.GND2, IC2.GND3, IC2.GND4, R1.2, X1.1, X1.10
- net P8.13: now also BB.CAPE2B.EHRPWM.2B; no longer BB.CAPE1B.EHRPWM.2B
- net P8.14: now also BB.CAPE2B.GPIO26; no longer BB.CAPE1B.GPIO26
- net P8.15: now also BB.CAPE2B.GPIO47; no longer BB.CAPE1B.GPIO47
- net P8.16: now also BB.CAPE2B.GPIO46; no longer BB.CAPE1B.GPIO46
- net P8.17: now also BB.CAPE2B.GPIO27; no longer BB.CAPE1B.GPIO27
- net P8.18: now also BB.CAPE2B.GPIO65; no longer BB.CAPE1B.GPIO65
- net P8.19: now also BB.CAPE2B.EHRPWM.2A; no longer BB.CAPE1B.EHRPWM.2A
- net P8.20: now also BB.CAPE2B.MMC1.CMD; no longer BB.CAPE1B.MMC1.CMD
- net P8.21: now also BB.CAPE2B.MMC1.CLK; no longer BB.CAPE1B.MMC1.CLK
- net P8.22: now also BB.CAPE2B.MMC1.DAT5; no longer BB.CAPE1B.MMC1.DAT5
- net P8.23: now also BB.CAPE2B.MMC1.DAT4; no longer BB.CAPE1B.MMC1.DAT4
- net P8.24: now also BB.CAPE2B.MMC1.DAT1; no longer BB.CAPE1B.MMC1.DAT1
- net P8.25: now also BB.CAPE2B.MMC1.DAT0; no longer BB.CAPE1B.MMC1.DAT0
- net P8.26: now also BB.CAPE2B.GPIO61; no longer BB.CAPE1B.GPIO61
- net P8.27: now also BB.CAPE2B.LCD.VSYNC; no longer BB.CAPE1B.LCD.VSYNC
- net P8.28: now also BB.CAPE2B.LCD.PCLK; no longer BB.CAPE1B.LCD.PCLK
- net P8.29: now also BB.CAPE2B.LCD.HSYNC; no longer BB.CAPE1B.LCD.HSYNC
- net P8.3: now also BB.CAPE2B.MMC1.DAT6; no longer BB.CAPE1B.MMC1.DAT6
- net P8.30: now also BB.CAPE2B.LCD.AC.BIAS; no longer BB.CAPE1B.LCD.AC.BIAS
- net P8.31: now also BB.CAPE2B.LCD.DATA14; no longer BB.CAPE1B.LCD.DATA14
- net P8.32: now also BB.CAPE2B.LCD.DATA15; no longer BB.CAPE1B.LCD.DATA15
- net P8.33: now also BB.CAPE2B.LCD.DATA13; no longer BB.CAPE1B.LCD.DATA13
- net P8.34: now also BB.CAPE2B.LCD.DATA11; no longer BB.CAPE1B.LCD.DATA11
- net P8.35: now also BB.CAPE2B.LCD.DATA12; no longer BB.CAPE1B.LCD.DATA12
- net P8.36: now also BB.CAPE2B.LCD.DATA10; no longer BB.CAPE1B.LCD.DATA10
- net P8.37: now also BB.CAPE2B.LCD.DATA8; no longer BB.CAPE1B.LCD.DATA8
- net P8.38: now also BB.CAPE2B.LCD.DATA9; no longer BB.CAPE1B.LCD.DATA9
- net P8.39: now also BB.CAPE2B.LCD.DATA6; no longer BB.CAPE1B.LCD.DATA6
- net P8.4: now also BB.CAPE2B.MMC1.DAT7; no longer BB.CAPE1B.MMC1.DAT7
- net P8.40: now also BB.CAPE2B.LCD.DATA7; no longer BB.CAPE1B.LCD.DATA7
- net P8.41: now also BB.CAPE2B.LCD.DATA4; no longer BB.CAPE1B.LCD.DATA4
- net P8.42: now also BB.CAPE2B.LCD.DATA5; no longer BB.CAPE1B.LCD.DATA5
- net P8.43: now also BB.CAPE2B.LCD.DATA2; no longer BB.CAPE1B.LCD.DATA2
- net P8.44: now also BB.CAPE2B.LCD.DATA3; no longer BB.CAPE1B.LCD.DATA3
- net P8.45: now also BB.CAPE2B.LCD.DATA0; no longer BB.CAPE1B.LCD.DATA0
- net P8.46: now also BB.CAPE2B.LCD.DATA1; no longer BB.CAPE1B.LCD.DATA1
- net P8.5: now also BB.CAPE2B.MMC1.DAT2; no longer BB.CAPE1B.MMC1.DAT2
- net P8.6: now also BB.CAPE2B.MMC1.DAT3; no longer BB.CAPE1B.MMC1.DAT3
- net P8.7: now also BB.CAPE2B.GPIO66; no longer BB.CAPE1B.GPIO66
- net P8.8: now also BB.CAPE2B.GPIO67; no longer BB.CAPE1B.GPIO67
- net P8.9: now also BB.CAPE2B.GPIO69; no longer BB.CAPE1B.GPIO69
- net P9.11: now also BB.CAPE2A.UART4.RXD; no longer BB.CAPE1A.UART4.RXD
- net P9.12: now also BB.CAPE2A.GPIO60; no longer BB.CAPE1A.GPIO60
- net P9.13: now also BB.CAPE2A.UART4.TXD; no longer BB.CAPE1A.UART4.TXD
- net P9.14: now also BB.CAPE2A.EHRPWM.1A; no longer BB.CAPE1A.EHRPWM.1A
- net P9.15: now also BB.CAPE2A.GPIO48; no longer BB.CAPE1A.GPIO48
- net P9.16: now also BB.CAPE2A.EHRPWM.1B; no longer BB.CAPE1A.EHRPWM.1B
- net P9.17: now also BB.CAPE2A.SPI0.CS0; no longer BB.CAPE1A.SPI0.CS0
- net P9.18: now also BB.CAPE2A.SPI0.D1; no longer BB.CAPE1A.SPI0.D1
- net P9.21: now also BB.CAPE2A.SPI0.D0; no longer BB.CAPE1A.SPI0.D0
- net P9.22: now also BB.CAPE2A.SPI0.SCK; no longer BB.CAPE1A.SPI0.SCK
- net P9.23: now also BB.CAPE2A.GPIO49; no longer BB.CAPE1A.GPIO49
- net P9.24: now also BB.CAPE2A.UART1.TXD; no longer BB.CAPE1A.UART1.TXD
- net P9.25: now also BB.CAPE2A.GPIO117; no longer BB.CAPE1A.GPIO117
- net P9.26: now also BB.CAPE2A.UART1.RXD; no longer BB.CAPE1A.UART1.RXD
- net P9.28: now also BB.CAPE2A.SPI1.CS0; no longer BB.CAPE1A.SPI1.CS0
- net P9.29: now also BB.CAPE2A.SPI1.D0; no longer BB.CAPE1A.SPI1.D0
- net P9.31: now also BB.CAPE2A.SPI1.SCK; no longer BB.CAPE1A.SPI1.SCK
- net P9.32: now also BB.CAPE2A.AVDD.ADC; no longer BB.CAPE1A.AVDD.ADC
- net P9.33: now also BB.CAPE2A.AIN4; no longer BB.CAPE1A.AIN4
- net P9.34: now also BB.CAPE2A.AGND.ADC; no longer BB.CAPE1A.AGND.ADC
- net P9.35: now also BB.CAPE2A.AIN6; no longer BB.CAPE1A.AIN6
- net P9.36: now also BB.CAPE2A.AIN5; no longer BB.CAPE1A.AIN5
- net P9.37: now also BB.CAPE2A.AIN2; no longer BB.CAPE1A.AIN2
- net P9.38: now also BB.CAPE2A.AIN3; no longer BB.CAPE1A.AIN3
- net P9.39: now also BB.CAPE2A.AIN0; no longer BB.CAPE1A.AIN0
- net P9.40: now also BB.CAPE2A.AIN1; no longer BB.CAPE1A.AIN1
- net VCC: now also BB.CAPE2A.VDD.3V3(1), BB.CAPE2A.VDD.3V3(2), C1.1, C2.1, R1.1, R10.2, R11.2, R12.2, R2.1, R3.1, R4.1, R5.1, R6.1, R9.1, SJ1.1, SJ2.1, U1.VCC, U2.VDD; no longer BB.CAPE1A.VDD.3V3(1), BB.CAPE1A.VDD.3V3(2), X1.5
- net VIN: now also S1.2, S10.2, S11.2, S12.2, S13.2, S14.2, S15.2, S16.2, S2.2, S3.2, S4.2, S5.2, S6.2, S7.2, S8.2, S9.2, X1.1; no longer C1.+, D1.A, X1.9
Other:
- note added: "------------------------------"
- note added: "1 | 0 | 1 | 0 | A2 | A1 | A0 | R/W"
- note added: "1 | 0 | 1 | 0 | H | H | H | R/W = 0x57"
- note added: "1 | 0 | 1 | 0 | H | H | L | R/W = 0x56"
- note added: "1 | 0 | 1 | 0 | H | L | H | R/W = 0x55"
- note added: "1 | 0 | 1 | 0 | H | L | L | R/W = 0x54"
- note added: "1 | 0 | 1 | 0 | L | H | H | R/W = 0x53"
- note added: "1 | 0 | 1 | 0 | L | H | L | R/W = 0x52"
- note added: "1 | 0 | 1 | 0 | L | L | H | R/W = 0x51"
- note added: "1 | 0 | 1 | 0 | L | L | L | R/W = 0x50"
- note added: "BeagleBone Headers and EEPROM"
- note added: "PWM Driver and Headers"
- note added: "Slave Address: 1 | A5 | A4 | A3 | A2 | A1 | A0 1 | 1 | 1 | 1 | 1 | 1 | 1"
- note removed: "BeagleBone Headers"
- note removed: "Power"
- note removed: "Power ICs and Header"
- moved on the sheet: R1, R2, R3
