File: designs/Comms/Comms_Cape.brd (EAGLE design)
At the start: 71.8 x 58.4 mm, 36 parts, among them IC2 74LVC1G57, IC3 MAX13487EESA, IC4 SN65HVD230, T1 PBSS4350Z 50V 3A, T2 PBSS4350Z 50V 3A

Commit message: Merge Comms cape updates
Parts:
- added FUD4, FUD5, FUD6: FIDUCIAL, GHI:FIDUCIAL_40MIL
- moved C1 15.4 mm to (28.8, 15.6), turned to 90 degrees
- moved R4 15.0 mm to (28.8, 13.5), turned to 90 degrees
- moved R6 9.63 mm to (29.3, 10.3), turned to 0 degrees
- moved IC1 8.67 mm to (25.7, 14.2), turned to 90 degrees
- moved SJ1 6.27 mm to (18.4, 15.0), turned to 0 degrees
- moved SJ2 5.89 mm to (18.4, 13.5), turned to 0 degrees
- moved R5 5.76 mm to (26.7, 10.3), turned to 180 degrees
- moved R3 3.14 mm to (22.9, 13.5), turned to 90 degrees
- moved R1 2.17 mm to (20.3, 13.5), turned to 90 degrees
- moved R2 0.92 mm to (21.6, 13.5), turned to 90 degrees
- renumbered BB.CAPE1 to BB.CAPE2
Connections:
- new net AGND: BB.CAPE2.B9.34, BB.CAPE2.T9.34, R10.1, R9.1
- new net P8.10: BB.CAPE2.B8.10, BB.CAPE2.T8.10
- new net P8.11: BB.CAPE2.B8.11, BB.CAPE2.T8.11
- new net P8.12: BB.CAPE2.B8.12, BB.CAPE2.T8.12
- new net P8.13: BB.CAPE2.B8.13, BB.CAPE2.T8.13
- new net P8.14: BB.CAPE2.B8.14, BB.CAPE2.T8.14
- new net P8.15: BB.CAPE2.B8.15, BB.CAPE2.T8.15
- new net P8.16: BB.CAPE2.B8.16, BB.CAPE2.T8.16
- new net P8.17: BB.CAPE2.B8.17, BB.CAPE2.T8.17
- new net P8.18: BB.CAPE2.B8.18, BB.CAPE2.T8.18
- new net P8.19: BB.CAPE2.B8.19, BB.CAPE2.T8.19
- new net P8.20: BB.CAPE2.B8.20, BB.CAPE2.T8.20
- new net P8.21: BB.CAPE2.B8.21, BB.CAPE2.T8.21
- new net P8.22: BB.CAPE2.B8.22, BB.CAPE2.T8.22
- new net P8.23: BB.CAPE2.B8.23, BB.CAPE2.T8.23
- new net P8.24: BB.CAPE2.B8.24, BB.CAPE2.T8.24
- new net P8.25: BB.CAPE2.B8.25, BB.CAPE2.T8.25
- new net P8.26: BB.CAPE2.B8.26, BB.CAPE2.T8.26
- new net P8.27: BB.CAPE2.B8.27, BB.CAPE2.T8.27
- new net P8.28: BB.CAPE2.B8.28, BB.CAPE2.T8.28
- new net P8.29: BB.CAPE2.B8.29, BB.CAPE2.T8.29
- new net P8.3: BB.CAPE2.B8.3, BB.CAPE2.T8.3
- new net P8.30: BB.CAPE2.B8.30, BB.CAPE2.T8.30
- new net P8.31: BB.CAPE2.B8.31, BB.CAPE2.T8.31
- new net P8.32: BB.CAPE2.B8.32, BB.CAPE2.T8.32
- new net P8.33: BB.CAPE2.B8.33, BB.CAPE2.T8.33
- new net P8.34: BB.CAPE2.B8.34, BB.CAPE2.T8.34
- new net P8.35: BB.CAPE2.B8.35, BB.CAPE2.T8.35
- new net P8.36: BB.CAPE2.B8.36, BB.CAPE2.T8.36
- new net P8.37: BB.CAPE2.B8.37, BB.CAPE2.T8.37
- new net P8.38: BB.CAPE2.B8.38, BB.CAPE2.T8.38
- new net P8.39: BB.CAPE2.B8.39, BB.CAPE2.T8.39
- new net P8.4: BB.CAPE2.B8.4, BB.CAPE2.T8.4
- new net P8.40: BB.CAPE2.B8.40, BB.CAPE2.T8.40
- new net P8.41: BB.CAPE2.B8.41, BB.CAPE2.T8.41
- new net P8.42: BB.CAPE2.B8.42, BB.CAPE2.T8.42
- new net P8.43: BB.CAPE2.B8.43, BB.CAPE2.T8.43
- new net P8.44: BB.CAPE2.B8.44, BB.CAPE2.T8.44
- new net P8.45: BB.CAPE2.B8.45, BB.CAPE2.T8.45
- new net P8.46: BB.CAPE2.B8.46, BB.CAPE2.T8.46
- new net P8.5: BB.CAPE2.B8.5, BB.CAPE2.T8.5
- new net P8.6: BB.CAPE2.B8.6, BB.CAPE2.T8.6
- new net P8.7: BB.CAPE2.B8.7, BB.CAPE2.T8.7
- new net P8.8: BB.CAPE2.B8.8, BB.CAPE2.T8.8
- new net P8.9: BB.CAPE2.B8.9, BB.CAPE2.T8.9
- new net P9.10: BB.CAPE2.B9.10, BB.CAPE2.T9.10
- new net P9.12: BB.CAPE2.B9.12, BB.CAPE2.T9.12
- new net P9.14: BB.CAPE2.B9.14, BB.CAPE2.T9.14
- new net P9.16: BB.CAPE2.B9.16, BB.CAPE2.T9.16
- new net P9.17: BB.CAPE2.B9.17, BB.CAPE2.T9.17
- new net P9.18: BB.CAPE2.B9.18, BB.CAPE2.T9.18
- new net P9.21: BB.CAPE2.B9.21, BB.CAPE2.T9.21
- new net P9.22: BB.CAPE2.B9.22, BB.CAPE2.T9.22
- new net P9.25: BB.CAPE2.B9.25, BB.CAPE2.T9.25
- new net P9.27: BB.CAPE2.B9.27, BB.CAPE2.T9.27
- new net P9.28: BB.CAPE2.B9.28, BB.CAPE2.T9.28
- new net P9.29: BB.CAPE2.B9.29, BB.CAPE2.T9.29
- new net P9.30: BB.CAPE2.B9.30, BB.CAPE2.T9.30
- new net P9.31: BB.CAPE2.B9.31, BB.CAPE2.T9.31
- new net P9.32: BB.CAPE2.B9.32, BB.CAPE2.T9.32
- new net P9.33: BB.CAPE2.B9.33, BB.CAPE2.T9.33
- new net P9.37: BB.CAPE2.B9.37, BB.CAPE2.T9.37
- new net P9.38: BB.CAPE2.B9.38, BB.CAPE2.T9.38
- new net P9.39: BB.CAPE2.B9.39, BB.CAPE2.T9.39
- new net P9.40: BB.CAPE2.B9.40, BB.CAPE2.T9.40
- new net P9.41: BB.CAPE2.B9.41, BB.CAPE2.T9.41
- new net P9.42: BB.CAPE2.B9.42, BB.CAPE2.T9.42
- new net P9.9: BB.CAPE2.B9.9, BB.CAPE2.T9.9
- net GND: now also R1.1; no longer R10.1, R9.1, SJ1.1
- net SINK.A: now also BB.CAPE2.B9.15, BB.CAPE2.T9.15; no longer BB.CAPE2.B9.25, BB.CAPE2.T9.25
- net SINK.B: now also BB.CAPE2.B9.23, BB.CAPE2.T9.23; no longer BB.CAPE2.B9.27, BB.CAPE2.T9.27
- net VCC: now also SJ1.1; no longer R1.1
Routing:
- net AGND: track 0.00 -> 32.7 mm, vias 0 -> 3
- net WP: track 17.4 -> 36.0 mm
- net SDA: track 24.9 -> 9.50 mm, vias 3 -> 1
- net SCL: track 29.1 -> 14.7 mm, vias 3 -> 1
- net SINK.A: track 27.1 -> 39.1 mm
- net P8.8: track 0.00 -> 3.47 mm, vias 0 -> 1
- net P8.6: track 0.00 -> 3.47 mm, vias 0 -> 1
- net P8.46: track 0.00 -> 3.47 mm, vias 0 -> 1
- net P8.44: track 0.00 -> 3.47 mm, vias 0 -> 1
- net P8.42: track 0.00 -> 3.47 mm, vias 0 -> 1
- net P8.40: track 0.00 -> 3.47 mm, vias 0 -> 1
- net P8.4: track 0.00 -> 3.47 mm, vias 0 -> 1
- net P8.38: track 0.00 -> 3.47 mm, vias 0 -> 1
- net P8.36: track 0.00 -> 3.47 mm, vias 0 -> 1
- net P8.34: track 0.00 -> 3.47 mm, vias 0 -> 1
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Other:
- board text added: "A2"
- board text added: "Comms"
- board text added: "IO48"
- board text added: "IO49"
- board text removed: "COM"
- board text removed: "IO115"
- board text removed: "IO117"
- board text removed: "Industrial"
