File: designs/Comms/Comms_Cape.sch (EAGLE design)
At the start: 36 parts, among them IC2 74LVC1G57, IC3 MAX13487EESA, IC4 SN65HVD230, T1 PBSS4350Z 50V 3A, T2 PBSS4350Z 50V 3A

Commit message: Merge Comms cape updates
Parts:
- removed BB.CAPE1: BEAGLEBONE.CAPE.TOP/BOTTOM-PADS, GHI-Solutions:BEAGLEBONE.CAPE.TOP/BOTTOM-PADS
- added BB.CAPE2: BEAGLEBONE.CAPE.TOP/BOTTOM-PADS, GHI-Solutions:BEAGLEBONE.CAPE.TOP/BOTTOM-PADS
- added FUD4, FUD5, FUD6: FIDUCIAL, GHI:FIDUCIAL
Connections:
- new net AGND: BB.CAPE2A.AGND.ADC, R10.1, R9.1
- new net P8.10: BB.CAPE2B.GPIO68
- new net P8.11: BB.CAPE2B.GPIO45
- new net P8.12: BB.CAPE2B.GPIO44
- new net P8.13: BB.CAPE2B.EHRPWM.2B
- new net P8.14: BB.CAPE2B.GPIO26
- new net P8.15: BB.CAPE2B.GPIO47
- new net P8.16: BB.CAPE2B.GPIO46
- new net P8.17: BB.CAPE2B.GPIO27
- new net P8.18: BB.CAPE2B.GPIO65
- new net P8.19: BB.CAPE2B.EHRPWM.2A
- new net P8.20: BB.CAPE2B.MMC1.CMD
- new net P8.21: BB.CAPE2B.MMC1.CLK
- new net P8.22: BB.CAPE2B.MMC1.DAT5
- new net P8.23: BB.CAPE2B.MMC1.DAT4
- new net P8.24: BB.CAPE2B.MMC1.DAT1
- new net P8.25: BB.CAPE2B.MMC1.DAT0
- new net P8.26: BB.CAPE2B.GPIO61
- new net P8.27: BB.CAPE2B.LCD.VSYNC
- new net P8.28: BB.CAPE2B.LCD.PCLK
- new net P8.29: BB.CAPE2B.LCD.HSYNC
- new net P8.3: BB.CAPE2B.MMC1.DAT6
- new net P8.30: BB.CAPE2B.LCD.AC.BIAS
- new net P8.31: BB.CAPE2B.LCD.DATA14
- new net P8.32: BB.CAPE2B.LCD.DATA15
- new net P8.33: BB.CAPE2B.LCD.DATA13
- new net P8.34: BB.CAPE2B.LCD.DATA11
- new net P8.35: BB.CAPE2B.LCD.DATA12
- new net P8.36: BB.CAPE2B.LCD.DATA10
- new net P8.37: BB.CAPE2B.LCD.DATA8
- new net P8.38: BB.CAPE2B.LCD.DATA9
- new net P8.39: BB.CAPE2B.LCD.DATA6
- new net P8.4: BB.CAPE2B.MMC1.DAT7
- new net P8.40: BB.CAPE2B.LCD.DATA7
- new net P8.41: BB.CAPE2B.LCD.DATA4
- new net P8.42: BB.CAPE2B.LCD.DATA5
- new net P8.43: BB.CAPE2B.LCD.DATA2
- new net P8.44: BB.CAPE2B.LCD.DATA3
- new net P8.45: BB.CAPE2B.LCD.DATA0
- new net P8.46: BB.CAPE2B.LCD.DATA1
- new net P8.5: BB.CAPE2B.MMC1.DAT2
- new net P8.6: BB.CAPE2B.MMC1.DAT3
- new net P8.7: BB.CAPE2B.GPIO66
- new net P8.8: BB.CAPE2B.GPIO67
- new net P8.9: BB.CAPE2B.GPIO69
- new net P9.10: BB.CAPE2A.SYS.RESET#
- new net P9.12: BB.CAPE2A.GPIO60
- new net P9.14: BB.CAPE2A.EHRPWM.1A
- new net P9.16: BB.CAPE2A.EHRPWM.1B
- new net P9.17: BB.CAPE2A.SPI0.CS0
- new net P9.18: BB.CAPE2A.SPI0.D1
- new net P9.21: BB.CAPE2A.SPI0.D0
- new net P9.22: BB.CAPE2A.SPI0.SCK
- new net P9.25: BB.CAPE2A.GPIO117
- new net P9.27: BB.CAPE2A.GPIO115
- new net P9.28: BB.CAPE2A.SPI1.CS0
- new net P9.29: BB.CAPE2A.SPI1.D0
- new net P9.30: BB.CAPE2A.GPIO112
- new net P9.31: BB.CAPE2A.SPI1.SCK
- new net P9.32: BB.CAPE2A.AVDD.ADC
- new net P9.33: BB.CAPE2A.AIN4
- new net P9.37: BB.CAPE2A.AIN2
- new net P9.38: BB.CAPE2A.AIN3
- new net P9.39: BB.CAPE2A.AIN0
- new net P9.40: BB.CAPE2A.AIN1
- new net P9.41: BB.CAPE2A.GPIO20
- new net P9.42: BB.CAPE2A.ECAPPWM0
- new net P9.9: BB.CAPE2A.PWR.BTN
- net +5V: now also BB.CAPE2A.VDD.5V(1), BB.CAPE2A.VDD.5V(2); no longer BB.CAPE1A.VDD.5V(1), BB.CAPE1A.VDD.5V(2)
- net 4-20MA.LOOP.A: now also BB.CAPE2A.AIN5; no longer BB.CAPE1A.AIN5
- net 4-20MA.LOOP.B: now also BB.CAPE2A.AIN6; no longer BB.CAPE1A.AIN6
- net CAN.RD: now also BB.CAPE2A.UART1.TXD; no longer BB.CAPE1A.UART1.TXD
- net CAN.TD: now also BB.CAPE2A.UART1.RXD; no longer BB.CAPE1A.UART1.RXD
- net GND: now also BB.CAPE2A.DGND1, BB.CAPE2A.DGND2, BB.CAPE2A.DGND3, BB.CAPE2A.DGND4, BB.CAPE2A.DGND5, BB.CAPE2A.DGND6, BB.CAPE2B.DGND1, BB.CAPE2B.DGND2, R1.1; no longer BB.CAPE1A.DGND1, BB.CAPE1A.DGND2, BB.CAPE1A.DGND3, BB.CAPE1A.DGND4, BB.CAPE1A.DGND5, BB.CAPE1A.DGND6, BB.CAPE1B.DGND1, BB.CAPE1B.DGND2, R10.1, R9.1, SJ1.1
- net RS485.RX: now also BB.CAPE2A.UART4.RXD; no longer BB.CAPE1A.UART4.RXD
- net RS485.TX: now also BB.CAPE2A.UART4.TXD; no longer BB.CAPE1A.UART4.TXD
- net SCL: now also BB.CAPE2A.I2C2.SCL; no longer BB.CAPE1A.I2C2.SCL
- net SDA: now also BB.CAPE2A.I2C2.SDA; no longer BB.CAPE1A.I2C2.SDA
- net SINK.A: now also BB.CAPE2A.GPIO48; no longer BB.CAPE1A.GPIO117
- net SINK.B: now also BB.CAPE2A.GPIO49; no longer BB.CAPE1A.GPIO115
- net SYS.VOUT: now also BB.CAPE2A.SYS.5V(1), BB.CAPE2A.SYS.5V(2); no longer BB.CAPE1A.SYS.5V(1), BB.CAPE1A.SYS.5V(2)
- net VCC: now also BB.CAPE2A.VDD.3V3(1), BB.CAPE2A.VDD.3V3(2), SJ1.1; no longer BB.CAPE1A.VDD.3V3(1), BB.CAPE1A.VDD.3V3(2), R1.1
Other:
- note added: "------------------------------"
- note added: "1 | 0 | 1 | 0 | A2 | A1 | A0 | R/W"
- note added: "1 | 0 | 1 | 0 | H | H | H | R/W = 0x57"
- note added: "1 | 0 | 1 | 0 | H | H | L | R/W = 0x56"
- note added: "1 | 0 | 1 | 0 | H | L | H | R/W = 0x55"
- note added: "1 | 0 | 1 | 0 | H | L | L | R/W = 0x54"
- note added: "1 | 0 | 1 | 0 | L | H | H | R/W = 0x53"
- note added: "1 | 0 | 1 | 0 | L | H | L | R/W = 0x52"
- note added: "1 | 0 | 1 | 0 | L | L | H | R/W = 0x51"
- note added: "1 | 0 | 1 | 0 | L | L | L | R/W = 0x50"
- note added: "A2"
- note added: "BeagleBone Headers and EEPROM"
- note added: "CAN and RS485 ICs and Sink transistors"
- moved on the sheet: C1, C2, C3, C4, IC1, IC2, IC3, IC4, JMP1, LED1, LED2, R1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
