File: designs/Display50/Display50_Cape.brd (EAGLE design)
At the start: 141 x 97.8 mm, 37 parts, among them IC1 PT4110, IC2 DNP (FAN5333BSX)

Commit message: Merge Display50 updates
Connections:
- removed net P8.9: BB.DISPLAY.CAPE-(BEAGLEBONE).B8.9, BB.DISPLAY.CAPE-(CAPE).B8.9
- removed net P9.12: BB.DISPLAY.CAPE-(BEAGLEBONE).B9.12, BB.DISPLAY.CAPE-(CAPE).B9.12
- new net P9.14: BB.DISPLAY.CAPE-(BEAGLEBONE).B9.14, BB.DISPLAY.CAPE-(CAPE).B9.14
- new net P9.30: BB.DISPLAY.CAPE-(BEAGLEBONE).B9.30, BB.DISPLAY.CAPE-(CAPE).B9.30
- net CAP.TOUCH.IRQ: now also BB.DISPLAY.CAPE-(BEAGLEBONE).B9.12, BB.DISPLAY.CAPE-(CAPE).B9.12; no longer BB.DISPLAY.CAPE-(BEAGLEBONE).B9.30, BB.DISPLAY.CAPE-(CAPE).B9.30
- net LCD.BACKLIGHT: now also BB.DISPLAY.CAPE-(BEAGLEBONE).B8.9, BB.DISPLAY.CAPE-(CAPE).B8.9; no longer BB.DISPLAY.CAPE-(BEAGLEBONE).B9.14, BB.DISPLAY.CAPE-(CAPE).B9.14
Routing:
- net P9.30: track 0.00 -> 139.6 mm, vias 0 -> 2
- net P9.14: track 0.00 -> 121.2 mm, vias 0 -> 2
- net P9.12: track 120.5 -> 0.00 mm, vias 2 -> 0
- net LCD.BACKLIGHT: track 156.4 -> 82.6 mm, vias 4 -> 3
- net P8.9: track 23.1 -> 0.00 mm
- net CAP.TOUCH.IRQ: track 177.8 -> 165.3 mm
- net P9.16: track 123.5 -> 122.7 mm
Other:
- board text added: "A2"
- board text added: "Display50"
- board text removed: "435"
- board text removed: "Display"
