File: designs/Display50/Display50_Cape.sch (EAGLE design)
At the start: 37 parts, among them IC1 PT4110, IC2 DNP (FAN5333BSX)

Commit message: Merge Display50 updates
Connections:
- removed net P8.9: BB.DISPLAY.CAPE-(BEAGLEBONE)B.GPIO69, BB.DISPLAY.CAPE-(CAPE)B.GPIO69
- removed net P9.12: BB.DISPLAY.CAPE-(BEAGLEBONE)A.GPIO60, BB.DISPLAY.CAPE-(CAPE)A.GPIO60
- new net P9.14: BB.DISPLAY.CAPE-(BEAGLEBONE)A.EHRPWM.1A, BB.DISPLAY.CAPE-(CAPE)A.EHRPWM.1A
- new net P9.30: BB.DISPLAY.CAPE-(BEAGLEBONE)A.GPIO112, BB.DISPLAY.CAPE-(CAPE)A.GPIO112
- net CAP.TOUCH.IRQ: now also BB.DISPLAY.CAPE-(BEAGLEBONE)A.GPIO60, BB.DISPLAY.CAPE-(CAPE)A.GPIO60; no longer BB.DISPLAY.CAPE-(BEAGLEBONE)A.GPIO112, BB.DISPLAY.CAPE-(CAPE)A.GPIO112
- net LCD.BACKLIGHT: now also BB.DISPLAY.CAPE-(BEAGLEBONE)B.GPIO69, BB.DISPLAY.CAPE-(CAPE)B.GPIO69; no longer BB.DISPLAY.CAPE-(BEAGLEBONE)A.EHRPWM.1A, BB.DISPLAY.CAPE-(CAPE)A.EHRPWM.1A
Other:
- note added: "------------------------------"
- note added: "1 | 0 | 1 | 0 | A2 | A1 | A0 | R/W"
- note added: "1 | 0 | 1 | 0 | H | H | H | R/W = 0x57"
- note added: "1 | 0 | 1 | 0 | H | H | L | R/W = 0x56"
- note added: "1 | 0 | 1 | 0 | H | L | H | R/W = 0x55"
- note added: "1 | 0 | 1 | 0 | H | L | L | R/W = 0x54"
- note added: "1 | 0 | 1 | 0 | L | H | H | R/W = 0x53"
- note added: "1 | 0 | 1 | 0 | L | H | L | R/W = 0x52"
- note added: "1 | 0 | 1 | 0 | L | L | H | R/W = 0x51"
- note added: "1 | 0 | 1 | 0 | L | L | L | R/W = 0x50"
- note added: "A2"
- note added: "Backlight Cap Touch LCD connector"
- note added: "BeagleBone Headers and EEPROM"
- moved on the sheet: 4.3, 5.0, BB.DISPLAY.CAPE-(BEAGLEBONE)A, BB.DISPLAY.CAPE-(BEAGLEBONE)B, BB.DISPLAY.CAPE-(CAPE)A, BB.DISPLAY.CAPE-(CAPE)B, C1, C2, C3, C4, C5, C6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
